File: HW/usb_relay_control/usb_relay_control.kicad_pcb (KiCad board)
At the start: 2 copper layers, 108 parts, among them IC1 LDL1117S33R, J1 8.06.04_J-LINK_NEEDLE_ADAPTER, J10 2301843-2, J2 USB_B_Micro, J3 Conn_01x03_Male, J4 Conn_01x04_Male, J5 Conn_01x05_Male, J6 Screw_Terminal_01x04, J7 Screw_Terminal_01x04, J8 Screw_Terminal_01x04, J9 Screw_Terminal_01x04, K1 SRD-05VDC-SL-C, K2 SRD-05VDC-SL-C, K3 SRD-05VDC-SL-C, K4 SRD-05VDC-SL-C, Q1 Q_NPN_BEC SMMBT3904LT1G, Q2 Q_NPN_BEC, Q3 Q_NPN_BEC, Q4 Q_NPN_BEC, SW1 SW_Push, SW2 SW_Push, U1 STM32F103CBTx, U2 INA4181A1IPWR, U3 TJA1051T-3, Y1 16 MHz Crystal

Commit message: ADD: AI antigravity review EMC according to IPC2221
Parts:
- removed D15: BZX84C3V3, Package_TO_SOT_SMD:SOT-23
- removed JP1: SolderJumper_3_Open, Jumper:SolderJumper-3_P1.3mm_Open_RoundedPad1.0x1.5mm_NumberLabels
- removed K3, K4: SRD-05VDC-SL-C, SRD-05VDC-SL-C:RELAY_SRD-05VDC-SL-C
- removed Q3, Q4: Q_NPN_BEC, Package_TO_SOT_SMD:SOT-23
- added C20: 0.1uF, Capacitor_SMD:C_0805_2012Metric, F.Cu at (217.1, 108.8)
- added C21: 4u7, Capacitor_SMD:C_0805_2012Metric, F.Cu at (193.7, 82.8)
- added C22: 4u7, Capacitor_SMD:C_0805_2012Metric, F.Cu at (186.3, 66.9)
- added C23: 10nF, Capacitor_SMD:C_0805_2012Metric, F.Cu at (252.8, 124.3)
- added C24: 0.1uF, Capacitor_SMD:C_0805_2012Metric, F.Cu at (187.8, 93.6)
- added C25: 0.1uF, Capacitor_SMD:C_0805_2012Metric, F.Cu at (196.8, 103.5)
- added C26: 10nF, Capacitor_SMD:C_0805_2012Metric, F.Cu at (182.2, 118.5)
- added C27: 0.1uF, Capacitor_SMD:C_0805_2012Metric, F.Cu at (193.4, 85.8)
- added C28: 0.1uF, Capacitor_SMD:C_0805_2012Metric, F.Cu at (184.1, 70.7)
- added C29: 0.1uF, Capacitor_SMD:C_0805_2012Metric, F.Cu at (191.4, 108.1)
- added C30: 0.1uF, Capacitor_SMD:C_0805_2012Metric, F.Cu at (185.7, 78.2)
- added C31: 10nF, Capacitor_SMD:C_0805_2012Metric, F.Cu at (212.8, 104.5)
- added C32: 10nF, Capacitor_SMD:C_0805_2012Metric, F.Cu at (234.8, 101.0)
- added C33: 10nF, Capacitor_SMD:C_0805_2012Metric, F.Cu at (240.0, 96.0)
- added C34: 47u, Capacitor_SMD:C_0805_2012Metric, F.Cu at (209.1, 70.0)
- added C35: 0.1uF, Capacitor_SMD:C_0805_2012Metric, F.Cu at (205.6, 70.0)
- added D18: PRTR5V0U2X, Package_TO_SOT_SMD:SOT-143, F.Cu at (167.2, 110.9)
- added D19: PRTR5V0U2X, Package_TO_SOT_SMD:SOT-143, F.Cu at (181.9, 76.6)
- added F2: 1A, Fuse:Fuse_0805_2012Metric, F.Cu at (182.0, 67.0)
- added F3: 1A, Fuse:Fuse_0805_2012Metric, F.Cu at (177.5, 116.4)
- added F4: 28mA, Fuse:Fuse_0603_1608Metric, F.Cu at (249.7, 94.6)
- added F5: 28mA, Fuse:Fuse_0603_1608Metric, F.Cu at (249.7, 92.2)
- added F6: 700mA, Fuse:Fuse_0603_1608Metric, F.Cu at (220.2, 52.0)
- added FID1: Fiducial, Fiducial:Fiducial_0.5mm_Mask1mm, F.Cu at (173.1, 138.0)
- added FID2: Fiducial, Fiducial:Fiducial_0.5mm_Mask1mm, F.Cu at (247.4, 138.0)
- added FID3: Fiducial, Fiducial:Fiducial_0.5mm_Mask1mm, F.Cu at (173.0, 52.1)
- added FID4: Fiducial, Fiducial:Fiducial_0.5mm_Mask1mm, F.Cu at (247.4, 52.2)
- added IC2: SIP32509DT-T1-GE3, SIP32509DT-T1-GE3:SOT95P284X110-6N, F.Cu at (193.0, 89.8)
- added IC3: SIP32509DT-T1-GE3, SIP32509DT-T1-GE3:SOT95P284X110-6N, F.Cu at (192.4, 78.7)
- added J11: USB_A, 292303-9:J_SMD_292303-9-4_2,2.5_14.85_14.06_8.9, F.Cu at (170.2, 83.8)
- added J12: USB_A, 292303-9:J_SMD_292303-9-4_2,2.5_14.85_14.06_8.9, F.Cu at (170.2, 102.2)
- added J13: Conn_01x03_Male, Connector_PinHeader_2.54mm:PinHeader_1x03_P2.54mm_Vertical, F.Cu at (229.7, 51.5)
- added J14: Conn_01x03_Male, Connector_PinHeader_2.54mm:PinHeader_1x03_P2.54mm_Vertical, F.Cu at (210.9, 51.8)
- added J15: Conn_01x03_Male, Connector_PinHeader_2.54mm:PinHeader_1x03_P2.54mm_Vertical, F.Cu at (175.6, 129.8)
- added J16: Conn_01x02_Male, Connector_PinHeader_2.54mm:PinHeader_1x02_P2.54mm_Vertical, F.Cu at (181.9, 138.3)
- added J17: Conn_01x03_Male, Connector_PinHeader_2.54mm:PinHeader_1x03_P2.54mm_Vertical, F.Cu at (216.4, 132.7)
- added J18: Conn_01x03_Male, Connector_PinHeader_2.54mm:PinHeader_1x03_P2.54mm_Vertical, F.Cu at (229.7, 54.6)
- added J19: Conn_01x05_Male, Connector_PinHeader_2.54mm:PinHeader_1x05_P2.54mm_Vertical, F.Cu at (250.3, 120.6)
- added J20: Conn_01x02_Male, Connector_PinHeader_2.54mm:PinHeader_1x02_P2.54mm_Vertical, F.Cu at (217.4, 138.6)
- added J21: Conn_01x02_Male, Connector_PinHeader_2.54mm:PinHeader_1x02_P2.54mm_Vertical, F.Cu at (221.2, 138.5)
- added J22: Screw_Terminal_01x02, footprints:CONN_OSTVN02A150_OST, F.Cu at (251.2, 100.7)
- added J23: Screw_Terminal_01x02, footprints:CONN_OSTVN02A150_OST, F.Cu at (251.2, 107.1)
- added R39: 10K, Resistor_SMD:R_0805_2012Metric, F.Cu at (245.3, 97.1)
- added R40: 10K, Resistor_SMD:R_0805_2012Metric, F.Cu at (245.2, 94.5)
- added R41: 0, Resistor_SMD:R_0805_2012Metric, F.Cu at (243.6, 91.3)
- added R42: 0, Resistor_SMD:R_0805_2012Metric, F.Cu at (168.2, 60.2)
- added R43: 0, Resistor_SMD:R_0805_2012Metric, F.Cu at (170.2, 127.0)
- added R44: 100K, Resistor_SMD:R_0805_2012Metric, F.Cu at (236.8, 92.7)
- added R45: 100K, Resistor_SMD:R_0805_2012Metric, F.Cu at (238.0, 106.3)
- added R46: 1k5, Resistor_SMD:R_0805_2012Metric, F.Cu at (241.3, 82.8)
- added U4: INA2181A1IDGSR, ul_INA2181A1IDGSR:INA2181A1IDGSR, F.Cu at (217.0, 112.5)
- C1, C2: value 10pF -> 8pF
- C11: value 1u -> 1uF
- C12, C13: value 10n -> 10nF
- C15, C17: value 100nF -> 0.1uF
- C16: value 100n -> 0.1uF
- C18: value 0.1u -> 0.1uF
- C19: value 4.7u -> 4.7nF
- C4, C5, C7, C8, C9: value 100n -> 10uF
- D1: value LED_Small -> RED LED
- D10: value LL4148 -> PRTR5V0U2X; footprint Diode_SMD:D_MiniMELF -> Package_TO_SOT_SMD:SOT-143
- D11: value LL4148 -> BZY55B3V3_RBG; footprint Diode_SMD:D_MiniMELF -> BZY55B3V3_RBG:BZY55B3V3RBG
- D12: value RED -> BZY55B3V3_RBG; footprint LED_SMD:LED_0805_2012Metric -> BZY55B3V3_RBG:BZY55B3V3RBG
- D13, D8: value RED -> RED LED
- D14: value BZX84C3V3 -> BZY55B3V3_RBG; footprint Package_TO_SOT_SMD:SOT-23 -> BZY55B3V3_RBG:BZY55B3V3RBG
- D16, D17: value BZX84C3V3 -> RED LED; footprint Package_TO_SOT_SMD:SOT-23 -> LED_SMD:LED_0805_2012Metric
- D2: value RED_LED -> RED LED
- D3: value GREEN_LED -> GREEN LED
- D4: value BLUE_LED -> BLUE LED
- D9: value RED -> PRTR5V0U2X; footprint LED_SMD:LED_0805_2012Metric -> Package_TO_SOT_SMD:SOT-143
- F1: value 2 A -> 1A
- IC1: footprint LDL1117s33:SOT230P700X180-4N -> LDL1117S33R:SOT230P700X180-4N
- J10: value 2301843-2 -> 2301843-1
- J2: value USB_B_Micro -> USB_B_Mini
- J3: footprint Connector_PinHeader_1.27mm:PinHeader_1x03_P1.27mm_Vertical -> Connector_PinHeader_2.54mm:PinHeader_1x03_P2.54mm_Vertical
- J4: value Conn_01x04_Male -> Conn_01x02_Male; footprint Connector_PinHeader_1.27mm:PinHeader_1x04_P1.27mm_Vertical -> Connector_PinHeader_2.54mm:PinHeader_1x02_P2.54mm_Vertical
- J5: footprint Connector_PinHeader_1.27mm:PinHeader_1x05_P1.27mm_Vertical -> Connector_PinHeader_2.54mm:PinHeader_1x05_P2.54mm_Vertical
- J8, J9: value Screw_Terminal_01x04 -> USB_B_Mini; footprint TerminalBlock_Phoenix:TerminalBlock_Phoenix_MKDS-1,5-4_1x04_P5.00mm_Horizontal -> Connector_USB:USB_Mini-B_Lumberg_2486_01_Horizontal
- Q1: value Q_NPN_BEC SMMBT3904LT1G -> Q_NPN_BEC MMBT3904-ND
- Q2: value Q_NPN_BEC -> MMBT3904-ND
- R1, R3: value 3.4k -> 332
- R10: value 60.4k -> 124k
- R11, R12: value 20k -> 47k
- R14, R28: value 10K -> 1K
- R16: value 1K -> 10
- R17: value 1K -> 1.78k
- R18: value 1K -> 10K
- R2, R6: value 10k -> 10K
- R20, R30: value 10K -> 10
- R21, R22: value 20m -> 32m; footprint Resistor_SMD:R_1020_2550Metric -> Resistor_SMD:R_2512_6332Metric
- R23: value 60.4k -> 1.78k
- R24: value 60.4k -> 10K
- R25, R26: value 20k -> 10K
- R29: value 1K -> 150
- R35, R36, R37, R38: value 10 -> 150
- R4: value 3.4k -> 300
- R5: value 3.4k -> 167
- R7: footprint Resistor_SMD:R_1020_2550Metric -> Resistor_SMD:R_2010_5025Metric
- R8: value 20m -> 124k; footprint Resistor_SMD:R_1020_2550Metric -> Resistor_SMD:R_0805_2012Metric
- R9: value 60.4k -> 20m; footprint Resistor_SMD:R_0805_2012Metric -> Resistor_SMD:R_2010_5025Metric
- U2: value INA4181A1IPWR -> INA2181A3QDGSRQ1; footprint INA4181A1IPWR:SOP65P640X120-20N -> ul_INA2181A3QDGSRQ1:INA2181A3QDGSRQ1
- moved J4 223.8 mm to (253.3, 94.6), turned to 180 degrees
- moved J7 220.2 mm to (228.4, 135.3)
- moved K2 211.8 mm to (236.0, 121.2)
- moved J1 200.1 mm to (248.1, 63.0)
- moved H2 197.8 mm to (250.0, 55.0)
- moved H4 193.9 mm to (250.0, 135.0)
- moved J6 193.3 mm to (193.5, 135.3)
- moved D7 187.0 mm to (217.8, 128.5), turned to 180 degrees
- moved FB2 184.8 mm to (244.3, 81.8), turned to 90 degrees
- moved R35 182.8 mm to (252.8, 127.8), turned to -90 degrees
- moved D13 182.2 mm to (247.2, 117.6), turned to -90 degrees
- moved R27 179.3 mm to (247.3, 122.0), turned to 180 degrees
- moved R12 177.7 mm to (247.5, 130.9), turned to 90 degrees
- moved C10 177.5 mm to (241.4, 77.2), turned to 90 degrees
- moved J5 177.4 mm to (253.2, 120.6), turned to 180 degrees
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Connections:
- D10 pad 1: +5V -> GND
- D10 pad 2: Net-(D10-Pad2) -> USB2_D-
- D11 pad 1: +5V -> Net-(D11-Pad1)
- D11 pad 2: Net-(D11-Pad2) -> GND
- D12 pad 1: Net-(D10-Pad2) -> Net-(D12-Pad1)
- D12 pad 2: Net-(D12-Pad2) -> GND
- D13 pad 1: Net-(D11-Pad2) -> Net-(D13-K)
- D13 pad 2: Net-(D13-Pad2) -> Net-(D13-A)
- D14 pad 1: GND -> Net-(D14-Pad1)
- D14 pad 2: unconnected-(D14-Pad2) -> GND
- D16 pad 2: unconnected-(D16-Pad2) -> Net-(D16-A)
- D17 pad 2: unconnected-(D17-Pad2) -> Net-(D17-A)
- D2 pad 1: RED_LED -> GND
- D3 pad 1: GREEN_LED -> GND
- D4 pad 1: BLUE_LED -> GND
- D6 pad 2: Net-(D6-Pad2) -> Net-(D13-K)
- D7 pad 2: Net-(D7-Pad2) -> Net-(D7-A)
- D8 pad 1: Net-(D6-Pad2) -> Net-(D7-A)
- D9 pad 1: Net-(D7-Pad2) -> GND
- D9 pad 2: Net-(D9-Pad2) -> USB1_D+
- J1 pad 8: unconnected-(J1-Pad8) -> JTDI
- J2 pad 6: unconnected-(J2-Pad6) -> Net-(J2-Shield)
- J3 pad 1: I2C_SDA -> GND
- J3 pad 2: I2C_SCK -> I2C_SDA
- J3 pad 3: GND -> I2C_SCK
- J4 pad 1: TEST_POINT0 -> Net-(J4-Pin_1)
- J4 pad 2: TEST_POINT1 -> Net-(J4-Pin_2)
- J5 pad 1: SPI_CS -> GND
- J5 pad 2: SPI_SCK -> SPI_CS
- J5 pad 3: SPI_SO -> SPI_SCK
- J5 pad 4: SPI_SIN -> SPI_MISO
- J5 pad 5: GND -> SPI_MOSI
- J6 pad 3: Net-(J6-Pad3) -> Net-(J6-Pin_3)
- J8 pad 1: SHUNT_3_M -> VBUS1_ESD
- J8 pad 2: Net-(J8-Pad2) -> USB1_D-
- J8 pad 3: Net-(J8-Pad3) -> USB1_D+
- J8 pad 4: GND -> unconnected-(J8-ID-Pad4)
- J9 pad 1: SHUNT_4_M -> VBUS2_ESD
- J9 pad 2: Net-(J9-Pad2) -> USB2_D-
- J9 pad 3: Net-(J9-Pad3) -> USB2_D+
- J9 pad 4: GND -> unconnected-(J9-ID-Pad4)
- K1 pad A1: Net-(D6-Pad2) -> Net-(D7-A)
- K1 pad NO: Net-(J6-Pad3) -> Net-(J6-Pin_3)
- K2 pad A1: Net-(D7-Pad2) -> Net-(D13-K)
- Q1 pad 1: Net-(Q1-Pad1) -> Net-(Q1-B)
- Q1 pad 3: Net-(D7-Pad2) -> Net-(D13-K)
- Q2 pad 1: Net-(Q2-Pad1) -> Net-(Q2-B)
- Q2 pad 3: Net-(D6-Pad2) -> Net-(D7-A)
- R13 pad 2: Net-(Q2-Pad1) -> RELAY_CONTROL_1
- R14 pad 1: GND -> Net-(Q2-B)
- R14 pad 2: Net-(Q1-Pad1) -> RELAY_CONTROL_2
- R16 pad 1: +5V -> EX_IN_ANALOG
- R16 pad 2: Net-(D9-Pad2) -> Net-(D11-Pad1)
- R17 pad 1: Net-(Q2-Pad1) -> VDD
- R17 pad 2: RELAY_CONTROL_2 -> Net-(J20-Pin_2)
- R18 pad 1: Net-(Q1-Pad1) -> Net-(J15-Pin_3)
- R18 pad 2: RELAY_CONTROL_1 -> VDD
- R19 pad 1: Net-(JP1-Pad1) -> GND
- R19 pad 2: VDD -> Net-(J15-Pin_3)
- R20 pad 1: GND -> VOLTAGE_SENSE_2
- R20 pad 2: Net-(JP1-Pad1) -> Net-(D12-Pad1)
- R21 pad 1: SHUNT_3_M -> SHUNT_4_P
- R21 pad 2: SHUNT_3_P -> SHUNT_4_M
- R22 pad 1: SHUNT_4_M -> SHUNT_3_P
- R22 pad 2: SHUNT_4_P -> SHUNT_3_M
- R23 pad 1: Net-(J8-Pad3) -> VDD
- R23 pad 2: VOLTAGE_SENSE_3 -> Net-(J21-Pin_2)
- R24 pad 1: Net-(J9-Pad3) -> GND
- R24 pad 2: VOLTAGE_SENSE_4 -> RELAY_CONTROL_2
- R25 pad 2: VOLTAGE_SENSE_3 -> RELAY_CONTROL_4
- R26 pad 2: VOLTAGE_SENSE_4 -> RELAY_CONTROL_3
- R27 pad 2: Net-(D12-Pad2) -> Net-(D13-A)
- R28 pad 1: GND -> Net-(Q1-B)
- R28 pad 2: Net-(Q3-Pad1) -> RELAY_CONTROL_1
- R29 pad 1: +5V -> MCU_EX_ANALOG_IN
- R29 pad 2: Net-(D13-Pad2) -> Net-(D11-Pad1)
- R3 pad 1: VDD -> RED_LED
- R30 pad 1: GND -> VOLTAGE_SENSE_1
- R30 pad 2: Net-(Q4-Pad1) -> Net-(D14-Pad1)
- R31 pad 1: Net-(Q3-Pad1) -> SHUNT_4_M
- R31 pad 2: RELAY_CONTROL_3 -> Net-(D16-A)
- R32 pad 1: Net-(Q4-Pad1) -> SHUNT_3_M
- R32 pad 2: RELAY_CONTROL_4 -> Net-(D17-A)
- R35 pad 1: CURRENT_SENSE_1 -> ADC_VOLTAGE_SENSE1
- R35 pad 2: Net-(U2-Pad2) -> Net-(D14-Pad1)
- R36 pad 1: CURRENT_SENSE_2 -> ADC_TEMP_SENS1
- R36 pad 2: Net-(U2-Pad8) -> EX_TEMP_SENS1
- R37 pad 1: CURRENT_SENSE_4 -> ADC_TEMP_SENS2
- R37 pad 2: Net-(U2-Pad19) -> EX_TEMP_SENS2
- R38 pad 1: CURRENT_SENSE_3 -> ADC_VOLTAGE_SENSE2
- R38 pad 2: Net-(U2-Pad13) -> Net-(D12-Pad1)
- R4 pad 1: VDD -> GREEN_LED
- R5 pad 1: VDD -> BLUE_LED
- R8 pad 1: SHUNT_1_M -> Net-(J6-Pin_3)
- R8 pad 2: SHUNT_1_P -> VOLTAGE_SENSE_2
- R9 pad 1: Net-(J6-Pad3) -> SHUNT_1_M
- R9 pad 2: VOLTAGE_SENSE_2 -> SHUNT_1_P
- U1 pad 10: CURRENT_SENSE_1 -> ADC_CURRENT_SENSE_1
- U1 pad 11: CURRENT_SENSE_2 -> ADC_CURRENT_SENSE_2
- U1 pad 12: CURRENT_SENSE_3 -> ADC_CURRENT_SENSE_3
- U1 pad 13: CURRENT_SENSE_4 -> ADC_CURRENT_SENSE_4
- U1 pad 14: VOLTAGE_SENSE_1 -> ADC_VOLTAGE_SENSE1
- U1 pad 15: VOLTAGE_SENSE_2 -> ADC_VOLTAGE_SENSE2
- U1 pad 16: VOLTAGE_SENSE_3 -> ADC_TEMP_SENS1
- U1 pad 17: VOLTAGE_SENSE_4 -> ADC_TEMP_SENS2
- U1 pad 18: TEST_POINT0 -> MCU_EX_ANALOG_IN
- U1 pad 19: TEST_POINT1 -> RELAY_CONTROL_3
- U1 pad 20: TEST_POINT2 -> RELAY_CONTROL_4
- U1 pad 29: RELAY_CONTROL_4 -> RELAY_CONTROL_1
- U1 pad 30: CAN_SILENCE -> RELAY_CONTROL_2
- U1 pad 31: unconnected-(U1-Pad31) -> PA10
- U1 pad 40: TEST_POINT3 -> PB4
- U1 pad 41: RELAY_CONTROL_1 -> CAN_SILENCE
- U1 pad 42: RELAY_CONTROL_2 -> UART_TX
- U1 pad 43: RELAY_CONTROL_3 -> UART_RX
- U2 pad 1: V_Ref -> ADC_CURRENT_SENSE_3
- U2 pad 10: unconnected-(U2-Pad10) -> VDD
- U2 pad 2: Net-(U2-Pad2) -> SHUNT_3_M
- U2 pad 3: SHUNT_1_M -> SHUNT_3_P
- U2 pad 4: SHUNT_1_P -> GND
- U2 pad 5: VDD -> GND
- U2 pad 6: SHUNT_2_P -> GND
- U2 pad 7: SHUNT_2_M -> SHUNT_4_P
- U2 pad 8: Net-(U2-Pad8) -> SHUNT_4_M
- U2 pad 9: V_Ref -> ADC_CURRENT_SENSE_4
Routing:
- net VDD: track 0.00 -> 347.6 mm, vias 0 -> 18
- net +5V: track 0.00 -> 204.1 mm, vias 0 -> 6
- net NRST: track 0.00 -> 97.6 mm, vias 0 -> 6
- net SHUNT_1_M: track 0.00 -> 75.9 mm, vias 0 -> 1
- net ADC_VOLTAGE_SENSE2: track 0.00 -> 62.2 mm, vias 0 -> 4
- net V_Ref_relay: track 0.00 -> 60.5 mm, vias 0 -> 1
- net VBUS1_ESD: track 0.00 -> 59.0 mm, vias 0 -> 4
- net SHUNT_4_M: track 0.00 -> 59.0 mm, vias 0 -> 4
- net EX_IN_ANALOG: track 0.00 -> 58.4 mm, vias 0 -> 4
- net I2C_SCK: track 0.00 -> 58.0 mm, vias 0 -> 1
- net USB1_D+: track 0.00 -> 54.9 mm, vias 0 -> 2
- net ADC_VOLTAGE_SENSE1: track 0.00 -> 54.8 mm
- net JTD0_TRACESWO: track 0.00 -> 54.4 mm, vias 0 -> 2
- net SHUNT_3_M: track 0.00 -> 51.2 mm, vias 0 -> 2
- net I2C_SDA: track 0.00 -> 50.6 mm, vias 0 -> 1
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- added copper zone on B.Cu, net GND
- added copper zone on F.Cu, net GND
- added copper zone on In1.Cu, net GND
- added copper zone on In2.Cu, net GND
Other:
- board outline added: 90 x 90 mm
- copper layers 2 -> 4
- board text added: "1V6"
- board text added: "3V3"
- board text added: "ADC"
- board text added: "AIN"
- board text added: "ANALOG_Input"
- board text added: "BOOT"
- board text added: "Bottom"
- board text added: "CAN"
- board text added: "COSMALLA"
- board text added: "CS"
- board text added: "GND"
- board text added: "I2C"
- board text added: "I2C_PULLUP"
- board text added: "IN1"
- board text added: "IN2"
- board text added: "Input"
- board text added: "MISO"
- board text added: "MOSI"
- board text added: "OUT1"
- board text added: "OUT2"
- board text added: "Out GPIOs"
- board text added: "Output"
- board text added: "PA10"
- board text added: "PB4"
- board text added: "RESET"
- board text added: "RX"
- board text added: "Relay1"
- board text added: "Relay2"
- board text added: "S/N:"
- board text added: "SCK"
- board text added: "SDA"
- board text added: "SPI"
- board text added: "TOP"
- board text added: "TX"
- board text added: "Thrm1"
- board text added: "Thrm2"
- board text added: "UART"
- board text added: "USB1 INPUT"
- board text added: "USB1 OUTPUT"
- board text added: "USB2 INPUT"
- board text added: "USB2 OUTPUT"
- board text added: "V 1.0"
- board text added: "VDD"
- board text added: "VDD_3V3"
- board text added: "Vref"
- board text added: "thrm"
