File: HW/usb_relay_control/usb_relay_control.kicad_sch (KiCad schematic)
At the start: 108 parts, among them IC1 LDL1117S33R, J1 8.06.04_J-LINK_NEEDLE_ADAPTER, J10 2301843-2, J2 USB_B_Micro, J3 Conn_01x03_Male, J4 Conn_01x04_Male, J5 Conn_01x05_Male, J6 Screw_Terminal_01x04, J7 Screw_Terminal_01x04, J8 Screw_Terminal_01x04, J9 Screw_Terminal_01x04, K1 SRD-05VDC-SL-C, K2 SRD-05VDC-SL-C, K3 SRD-05VDC-SL-C, K4 SRD-05VDC-SL-C, Q1 Q_NPN_BEC SMMBT3904LT1G, Q2 Q_NPN_BEC, Q3 Q_NPN_BEC, Q4 Q_NPN_BEC, SW1 SW_Push, SW2 SW_Push, U1 STM32F103CBTx, U2 INA4181A1IPWR, U3 TJA1051T-3, Y1 16 MHz Crystal

Commit message: ADD: AI antigravity review EMC according to IPC2221
Parts:
- removed D10, D11: LL4148, Diode_SMD:D_MiniMELF, symbol Diode:LL4148
- removed D12, D9: RED, LED_SMD:LED_0805_2012Metric, symbol Device:LED_Small
- removed D14, D15, D16, D17: BZX84C3V3, Package_TO_SOT_SMD:SOT-23, symbol Diode:BZX84Cxx
- removed D2: RED_LED, LED_SMD:LED_0805_2012Metric, symbol Device:LED_Small
- removed D3: GREEN_LED, LED_SMD:LED_0805_2012Metric, symbol Device:LED_Small
- removed D4: BLUE_LED, LED_SMD:LED_0805_2012Metric, symbol Device:LED_Small
- removed J4: Conn_01x04_Male, Connector_PinHeader_1.27mm:PinHeader_1x04_P1.27mm_Vertical, symbol Connector:Conn_01x04_Male
- removed J8, J9: Screw_Terminal_01x04, TerminalBlock_Phoenix:TerminalBlock_Phoenix_MKDS-1,5-4_1x04_P5.00mm_Horizontal, symbol Connector:Screw_Terminal_01x04
- removed JP1: SolderJumper_3_Open, Jumper:SolderJumper-3_P1.3mm_Open_RoundedPad1.0x1.5mm_NumberLabels, symbol Jumper:SolderJumper_3_Open
- removed K3, K4: SRD-05VDC-SL-C, SRD-05VDC-SL-C:RELAY_SRD-05VDC-SL-C, symbol SRD-05VDC-SL-C:SRD-05VDC-SL-C
- removed Q3, Q4: Q_NPN_BEC, Package_TO_SOT_SMD:SOT-23, symbol Device:Q_NPN_BEC
- removed U2: INA4181A1IPWR, INA4181A1IPWR:SOP65P640X120-20N, symbol INA4181A1IPWR:INA4181A1IPWR
- added C20, C24, C25, C27, C28, C29, C30, C70: 0.1uF, Capacitor_SMD:C_0805_2012Metric, symbol Device:C_Small
- added C21, C22: 4u7, Capacitor_SMD:C_0805_2012Metric, symbol Device:C_Small
- added C23, C26, C31, C32, C33: 10nF, Capacitor_SMD:C_0805_2012Metric, symbol Device:C_Small
- added C69: 47u, Capacitor_SMD:C_0805_2012Metric, symbol Device:C_Small
- added D10, D18, D19, D9: PRTR5V0U2X, Package_TO_SOT_SMD:SOT-143, symbol Power_Protection:PRTR5V0U2X
- added D11, D12, D14: BZY55B3V3_RBG, BZY55B3V3_RBG:BZY55B3V3RBG, symbol BZY55B3V3_RBG:BZY55B3V3_RBG
- added D16, D17: RED LED, LED_SMD:LED_0805_2012Metric, symbol Device:LED_Small
- added D2: RED LED, LED_SMD:LED_0805_2012Metric, symbol Device:LED
- added D3: GREEN LED, LED_SMD:LED_0805_2012Metric, symbol Device:LED
- added D4: BLUE LED, LED_SMD:LED_0805_2012Metric, symbol Device:LED
- added F2, F3: 1A, Fuse:Fuse_0805_2012Metric, symbol Device:Fuse_Small
- added F4, F5: 28mA, Fuse:Fuse_0603_1608Metric, symbol Device:Fuse_Small
- added F6: 700mA, Fuse:Fuse_0603_1608Metric, symbol Device:Fuse_Small
- added FID1, FID2, FID3, FID4: Fiducial, Fiducial:Fiducial_0.5mm_Mask1mm, symbol Mechanical:Fiducial
- added IC2, IC3: SIP32509DT-T1-GE3, SIP32509DT-T1-GE3:SOT95P284X110-6N, symbol SIP32509DT-T1-GE3:SIP32509DT-T1-GE3
- added J11, J12: USB_A, 292303-9:J_SMD_292303-9-4_2,2.5_14.85_14.06_8.9, symbol Connector:USB_A
- added J13, J14, J15, J17, J18: Conn_01x03_Male, Connector_PinHeader_2.54mm:PinHeader_1x03_P2.54mm_Vertical, symbol Connector:Conn_01x03_Male
- added J16, J20, J21, J4: Conn_01x02_Male, Connector_PinHeader_2.54mm:PinHeader_1x02_P2.54mm_Vertical, symbol Connector:Conn_01x02_Male
- added J19: Conn_01x05_Male, Connector_PinHeader_2.54mm:PinHeader_1x05_P2.54mm_Vertical, symbol Connector:Conn_01x05_Male
- added J22, J23: Screw_Terminal_01x02, footprints:CONN_OSTVN02A150_OST, symbol Connector:Screw_Terminal_01x02
- added J8, J9: USB_B_Mini, Connector_USB:USB_Mini-B_Lumberg_2486_01_Horizontal, symbol Connector:USB_B_Micro
- added R39, R40: 10K, Resistor_SMD:R_0805_2012Metric, symbol Device:R_Small
- added R41, R42, R43: 0, Resistor_SMD:R_0805_2012Metric, symbol Device:R_Small
- added R44, R45: 100K, Resistor_SMD:R_0805_2012Metric, symbol Device:R_Small
- added R46: 1k5, Resistor_SMD:R_0805_2012Metric, symbol Device:R_Small
- added U2: INA2181A3QDGSRQ1, ul_INA2181A3QDGSRQ1:INA2181A3QDGSRQ1, symbol 2023-02-03_08-27-06:INA2181A3QDGSRQ1
- added U4: INA2181A1IDGSR, ul_INA2181A1IDGSR:INA2181A1IDGSR, symbol 2023-02-03_08-18-01:INA2181A1IDGSR
- C1, C2: value 10pF -> 8pF
- C11: value 1u -> 1uF
- C12, C13: value 10n -> 10nF
- C15, C17: value 100nF -> 0.1uF
- C16: value 100n -> 0.1uF
- C18: value 0.1u -> 0.1uF
- C19: value 4.7u -> 4.7nF
- C4, C5, C7, C8, C9: value 100n -> 10uF
- D1: value LED_Small -> RED LED
- D13, D8: value RED -> RED LED
- F1: value 2 A -> 1A
- IC1: footprint LDL1117s33:SOT230P700X180-4N -> LDL1117S33R:SOT230P700X180-4N
- J10: value 2301843-2 -> 2301843-1
- J2: value USB_B_Micro -> USB_B_Mini
- J3: footprint Connector_PinHeader_1.27mm:PinHeader_1x03_P1.27mm_Vertical -> Connector_PinHeader_2.54mm:PinHeader_1x03_P2.54mm_Vertical
- J5: footprint Connector_PinHeader_1.27mm:PinHeader_1x05_P1.27mm_Vertical -> Connector_PinHeader_2.54mm:PinHeader_1x05_P2.54mm_Vertical
- Q1: value Q_NPN_BEC SMMBT3904LT1G -> Q_NPN_BEC MMBT3904-ND
- Q2: value Q_NPN_BEC -> MMBT3904-ND
- R1, R3: value 3.4k -> 332
- R10: value 60.4k -> 124k
- R11, R12: value 20k -> 47k
- R14, R28: value 10K -> 1K
- R16: value 1K -> 10
- R17: value 1K -> 1.78k
- R18: value 1K -> 10K
- R2, R6: value 10k -> 10K
- R20, R30: value 10K -> 10
- R21, R22: value 20m -> 32m; footprint Resistor_SMD:R_1020_2550Metric -> Resistor_SMD:R_2512_6332Metric
- R23: value 60.4k -> 1.78k
- R24: value 60.4k -> 10K
- R25, R26: value 20k -> 10K
- R29: value 1K -> 150
- R35, R36, R37, R38: value 10 -> 150
- R4: value 3.4k -> 300
- R5: value 3.4k -> 167
- R7: footprint Resistor_SMD:R_1020_2550Metric -> Resistor_SMD:R_2010_5025Metric
- R8: value 20m -> 124k; footprint Resistor_SMD:R_1020_2550Metric -> Resistor_SMD:R_0805_2012Metric
- R9: value 60.4k -> 20m; footprint Resistor_SMD:R_0805_2012Metric -> Resistor_SMD:R_2010_5025Metric
Connections:
- net SPI_SIN is gone; now on net SPI_MISO: J5.4 (Pin_4)
- net SPI_SO is gone; now on net SPI_SCK: J5.3 (Pin_3)
- net TEST_POINT1 is gone; now on net RELAY_CONTROL_3: U1.19 (PB1)
- net TEST_POINT2 is gone; now on net RELAY_CONTROL_4: U1.20 (PB2)
- net +5V: now also C69.1, C70.1; no longer R16.1, R29.1
- net BLUE_LED: now also R5.1
- net CAN_SILENCE: now also U1.41 (PB5); no longer U1.30 (PA9)
- net GND: now also J3.1 (Pin_1), J5.1 (Pin_1), R19.1, R24.1, C20.2, C21.2, C22.2, C23.1, C24.2, C25.2, C26.1, C27.2, C28.2, C29.2, C30.2, C31.1, C32.1, C33.1, C69.2, C70.2, D10.1 (GND), D11.2, D12.2, D14.2, D16.1 (K), D17.1 (K), D18.1 (GND), D19.1 (GND), D2.1 (K), D3.1 (K), D4.1 (K), D9.1 (GND), IC2.4 (GND), IC3.4 (GND), J11.4 (GND), J12.4 (GND), J13.1 (Pin_1), J15.1 (Pin_1), J16.1 (Pin_1), J17.1 (Pin_1), J18.1 (Pin_1), J19.1 (Pin_1), J8.5 (GND), J9.5 (GND), R39.2, R40.2, R41.1, R42.1, R43.1, R44.1, R45.1, U2.4 (GND), U2.5 (REF1), U2.6 (REF2), U4.4 (GND); no longer J3.3 (Pin_3), J5.5 (Pin_5), R14.1, R20.1, R28.1, R30.1
- net GREEN_LED: now also R4.1
- net I2C_SCK: now also J3.3 (Pin_3), J17.3 (Pin_3), J21.1 (Pin_1); no longer J3.2 (Pin_2)
- net I2C_SDA: now also J3.2 (Pin_2), J17.2 (Pin_2), J20.1 (Pin_1); no longer J3.1 (Pin_1)
- net JTDI: now also J1.8 (TDI)
- net RED_LED: now also R3.1
- net RELAY_CONTROL_1: now also R13.2, R28.2, U1.29 (PA8); no longer R18.2, U1.41 (PB5)
- net RELAY_CONTROL_2: now also R14.2, R24.2, U1.30 (PA9); no longer R17.2, U1.42 (PB6)
- net RELAY_CONTROL_3: now also R26.2, IC2.3 (EN); no longer R31.2, U1.43 (PB7)
- net RELAY_CONTROL_4: now also R25.2, IC3.3 (EN); no longer R32.2, U1.29 (PA8)
- net SHUNT_1_M: now also R9.1, U4.8 (IN-2); no longer R8.1
- net SHUNT_1_P: now also R9.2, U4.7 (IN+2); no longer R8.2
- net SHUNT_2_M: now also U4.2 (IN-1)
- net SHUNT_2_P: now also U4.3 (IN+1)
- net SHUNT_3_M: now also R22.2, R32.1, C29.1, D18.4 (VCC), J12.1 (VBUS), U2.2 (IN1-); no longer R21.1
- net SHUNT_3_P: now also R22.1, C24.1, IC2.1 (OUT_1), IC2.2 (OUT_2), U2.3 (IN1+); no longer R21.2
- net SHUNT_4_M: now also R21.2, R31.1, C30.1, D19.4 (VCC), J11.1 (VBUS), U2.8 (IN2-); no longer R22.1
- net SHUNT_4_P: now also R21.1, C25.1, IC3.1 (OUT_1), IC3.2 (OUT_2), U2.7 (IN2+); no longer R22.2
- net SPI_CS: now also J5.2 (Pin_2), J19.2 (Pin_2); no longer J5.1 (Pin_1)
- net SPI_MISO: now also J19.4 (Pin_4)
- net SPI_MOSI: now also J5.5 (Pin_5), J19.5 (Pin_5)
- net SPI_SCK: now also J19.3 (Pin_3); no longer J5.2 (Pin_2)
- net USB_D+: now also R46.2
- net VDD: now also R17.1, R18.2, R23.1, C20.1, F6.1, J22.2 (Pin_2), J23.2 (Pin_2), R46.1, U2.10 (VS), U4.10 (VS); no longer R19.2, R3.1, R4.1, R5.1
- net VOLTAGE_SENSE_1: now also R30.1; no longer U1.14 (PA4)
- net VOLTAGE_SENSE_2: now also R20.1, R8.2; no longer R9.2, U1.15 (PA5)
- net at K2.A1, Q1.3 (C): now also D13.1 (K), D6.2 (A); no longer D7.2 (A)
- net at R16.2: now also R29.2, D11.1
- net at D13.2 (A): now also R27.2; no longer R29.2
- net at R3.2: now also D2.2 (A)
- net at R38.2: now also R20.2, D12.1
- net EX_TEMP_SENS2: now reaches R37.2
- net EX_TEMP_SENS2: now also J23.1 (Pin_1), R45.2
- net at R35.2: now also R30.2, D14.1
- net EX_TEMP_SENS1: now reaches R36.2
- net EX_TEMP_SENS1: now also J22.1 (Pin_1), R44.2
- net at D8.1 (K), K1.A1, Q2.3 (C): now also D7.2 (A); no longer D6.2 (A)
- net at J6.3 (Pin_3), K1.NO: now also R8.1; no longer R9.1
- net at R5.2: now also D4.2 (A)
- net PA10: now reaches U1.31 (PA10)
- net PA10: now also F4.2, R39.1
- net at R4.2: now also D3.2 (A)
- net at J2.6 (Shield): now also R41.2
- net CURRENT_SENSE_1 renamed ADC_CURRENT_SENSE_1
- net ADC_CURRENT_SENSE_1: now also U4.9 (OUT2); no longer R35.1
- net CURRENT_SENSE_2 renamed ADC_CURRENT_SENSE_2
- net ADC_CURRENT_SENSE_2: now also U4.1 (OUT1); no longer R36.1
- net CURRENT_SENSE_3 renamed ADC_CURRENT_SENSE_3
- net ADC_CURRENT_SENSE_3: now also U2.1 (OUT1); no longer R38.1
- net CURRENT_SENSE_4 renamed ADC_CURRENT_SENSE_4
- net ADC_CURRENT_SENSE_4: now also U2.9 (OUT2); no longer R37.1
- net TEST_POINT0 renamed MCU_EX_ANALOG_IN
- net MCU_EX_ANALOG_IN: now also R29.1, C31.2
- net TEST_POINT3 renamed PB4
- net PB4: now also F5.2, R40.1
- removed net VOLTAGE_SENSE_3: R23.2, R25.2, U1.16 (PA6)
- removed net VOLTAGE_SENSE_4: R24.2, R26.2, U1.17 (PA7)
- new net: D17.2 (A), R32.2
- new net: J15.3 (Pin_3), R18.1, R19.2
- new net: Q1.1 (B), R28.1
- new net: F6.2, J14.1 (Pin_1), J14.2 (Pin_2), J14.3 (Pin_3)
- new net: Q2.1 (B), R14.1
- new net: J8.6 (Shield), R43.2
- new net: D16.2 (A), R31.2
- new net: F5.1, J4.2 (Pin_2)
- new net: J9.6 (Shield), R42.2
- new net: J21.2 (Pin_2), R23.2
- new net: F4.1, J4.1 (Pin_1)
- new net: J20.2 (Pin_2), R17.2
- new net ADC_TEMP_SENS1: C32.2, R36.1, U1.16 (PA6)
- new net ADC_TEMP_SENS2: C33.2, R37.1, U1.17 (PA7)
- new net ADC_VOLTAGE_SENSE1: C23.2, R35.1, U1.14 (PA4)
- new net ADC_VOLTAGE_SENSE2: C26.2, R38.1, U1.15 (PA5)
- new net EX_IN_ANALOG: J16.2 (Pin_2), R16.1
- new net UART_RX: J13.3 (Pin_3), J18.3 (Pin_3), U1.43 (PB7)
- new net UART_TX: J13.2 (Pin_2), J18.2 (Pin_2), U1.42 (PB6)
- new net USB1_D+: D18.2 (I/O1), D9.2 (I/O1), J12.3 (D+), J8.3 (D+)
- new net USB1_D-: D18.3 (I/O2), D9.3 (I/O2), J12.2 (D-), J8.2 (D-)
- new net USB2_D+: D10.3 (I/O2), D19.3 (I/O2), J11.3 (D+), J9.3 (D+)
- new net USB2_D-: D10.2 (I/O1), D19.2 (I/O1), J11.2 (D-), J9.2 (D-)
- new net VBUS1_ESD: C27.1, D9.4 (VCC), F3.1, J8.1 (VBUS)
- new net VBUS2_ESD: C28.1, D10.4 (VCC), F2.1, J9.1 (VBUS)
- new net VBUS_IN1: C21.1, F3.2, IC2.5 (IN_1), IC2.6 (IN_2)
- new net VBUS_IN2: C22.1, F2.2, IC3.5 (IN_1), IC3.6 (IN_2)
- new net V_Ref_relay: J15.2 (Pin_2), U4.5 (REF1), U4.6 (REF2)
- no-connect marks 15 -> 13
Other:
- note added: "100 uA Idle current"
- note added: "12/(124K+47K) = 70uA current for voltage sense"
- note added: "26 Volts max"
- note added: "5.5 volts MAX"
- note added: "70uA current for voltage sense"
- note added: "ADC Protection"
- note added: "D+ must pulled up to 1k5 resistor"
- note added: "EXTERNAL PIN HEADERS"
- note added: "External Analog Input"
- note added: "External VDD subbly"
- note added: "External thermistor sensor"
- note added: "F0603G0R02FNTR"
- note added: "F_CutOff = 1/(2(PI)(R)(C)) = 1/(2*3.14*(150+10)*10n) =~ 99.5KHz"
- note added: "Gain = 100"
- note added: "Gain = 20"
- note added: "I = 3 mA"
- note added: "J-Link Connector"
- note added: "Load Switch"
- note added: "MAX Current is 193mA + MCU current"
- note added: "MCU EXT. ANALOG IN 3V3 CUT AND FILTE"
- note added: "MMBT3904-ND BJT transistor: Ib(Sat) = 1mA , IC(Sat) = 10mA Ib = (3.3 - 0.7) / 1k = 2.6mA Ic1 = (5v- 2v - 0.2v ) / 1K = 3 mA Ic2 = 87 mA from coil circuit"
- note added: "RED led voltage drop = 2.2v GREEN led voltage drop = 2.4v BLUE led voltage drop = 2.8v"
- note added: "SF-0603S070-2"
- note added: "Supply 6 Volt max"
- note added: "USB connect indicator"
- note added: "USB connect-1A maximum"
- note added: "V_Out = (1A x 0.032 x 100) = 3.1 volts maximum"
- note added: "V_Out = (I_Load x R_Sense x GAIN) + V_Ref V_Out = (I_Load x R_Sense x 100) + V_Ref"
- note added: "Vin * (47/124+47) <= 3.3 V 12 Volt max"
- note added: "rated volts = 5.5V"
- note added: "the crystal load capacitance is 8pF, and assuming Cstray=4pF, then: CX1 = CX2 = 2(9pF - 5pF) = 8pF"
- note removed: "Iled ~1mA"
- note removed: "SMMBT3904LT1G BJT transistor: Ib(Sat) = 1mA , IC(Sat) = 10mA Ib = (3.3 - 0.7) / 1k = 2.6mA Ic = 5 / 1K = 5 mA"
- note removed: "the crystal load capacitance is 8pF, and assuming Cstray=3pF, then: CX1 = CX2 = 2(8pF - 3pF) = 10pF"
- company: QUANTTRONIX -> COSMALLA
- moved on the sheet: C14, C19, D5, J10, J3, J5, R33, R34, U3
